File: rk86kngmd.kicad_pcb (KiCad board)
At the start: 2 copper layers, 226.2 x 62.5 mm, 39 parts, among them P1 CONN_01X01, P10 CONN_01X01, P11 CONN_01X01, P12 CONN_01X01, P13 CONN_01X01, P14 CONN_01X01, P2 CONN_01X01, P3 CONN_01X01, P4 CONN_01X01, P5 CONN_01X01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

Commit message: Update
Parts:
- D1: footprint rk86ngmd:DIP-40-2.5mm -> rk86kngmd:DIP40-2.5mm
- moved D1 21.0 mm to (111.0, 81.8)
Routing:
- net /PC7: track 102.5 -> 182.3 mm, vias 3 -> 6
- net READY: track 62.7 -> 135.5 mm, vias 2 -> 5
- net RD_DATA: track 247.0 -> 174.2 mm, vias 13 -> 10
- net /D3: track 124.1 -> 77.3 mm, vias 7 -> 3
- net /D5: track 127.3 -> 94.3 mm, vias 4 -> 5

Commit message: Added credentials
Routing:
- net /PC7: track 182.3 -> 102.5 mm, vias 6 -> 3
- net READY: track 135.5 -> 62.7 mm, vias 5 -> 2
- net RD_DATA: track 174.2 -> 247.0 mm, vias 10 -> 13
- net /D3: track 77.3 -> 124.1 mm, vias 3 -> 7
- net /D5: track 94.3 -> 127.3 mm, vias 5 -> 4
Other:
- board text added: "2016 tnt23"
Changed lines of the file:
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@@
-(kicad_pcb (version 4) (host pcbnew 4.0.2+dfsg1-stable)
+(kicad_pcb (version 20170123) (host pcbnew "(2017-05-14 revision 14bb238b3)-makepkg")
   (general
     (links 219)
-    (no_connects 43)
-    (area 34.374999 68.8 267.300001 159.325)
+    (no_connects 0)
+    (area 34.374999 68.8 267.300001 159.4825)
     (thickness 1.6)
-    (drawings 14)
+    (drawings 15)
     (tracks 1209)
     (zones 0)
@@
       (hpglpenspeed 20)
       (hpglpendiameter 15)
-      (hpglpenoverlay 2)
       (psnegative false)
       (psa4output false)
@@
       (effects (font (size 1.5 1.5) (thickness 0.15)))
     )
-    (fp_text value К555ИР22 (at -4 4 360) (layer F.Fab)
+    (fp_text value К555ИР22 (at -4 4) (layer F.Fab)
       (effects (font (size 1.5 1.5) (thickness 0.15)))
     )
@@
       (effects (font (size 1.5 1.5) (thickness 0.15)))
     )
-    (fp_text value К555ИР13 (at -7.5 -5 360) (layer F.Fab)
+    (fp_text value К555ИР13 (at -7.5 -5) (layer F.Fab)
       (effects (font (size 1.5 1.5) (thickness 0.15)))
     )
@@
       (effects (font (size 1.5 1.5) (thickness 0.15)))
     )
-    (fp_text value К580ВВ55 (at 0 1.25 360) (layer F.Fab)
+    (fp_text value К580ВВ55 (at 0 1.25) (layer F.Fab)
       (effects (font (size 1.5 1.5) (thickness 0.15)))
     )
@@
       (net 12 "Net-(D1-Pad40)"))
   )
+  (gr_text "2016 tnt23" (at 251.59 119.335) (layer F.Cu)
+    (effects (font (size 1.5 1.5) (thickness 0.3)))
+  )
   (gr_line (start 124.75 133) (end 124.75 125.5) (layer Edge.Cuts) (width 0.1))
   (gr_line (start 48.5 125.5) (end 48.5 133) (layer Edge.Cuts) (width 0.1))
@@
   (segment (start 89.75 89.25) (end 89.75 93) (width 0.35) (layer F.Cu) (net 18) (status 10))
   (via (at 89.75 93) (size 1) (drill 0.5) (layers F.Cu B.Cu) (net 18))
-  (segment (start 136 98) (end 136 96.75) (width 0.35) (layer F.Cu) (net 18))
-  (segment (start 134.75 99.25) (end 136 98) (width 0.35) (layer F.Cu) (net 18))
-  (segment (start 134.75 108) (end 134.75 99.25) (width 0.35) (layer F.Cu) (net 18))
-  (segment (start 86 108) (end 134.75 108) (width 0.35) (layer B.Cu) (net 18))
-  (via (at 134.75 108) (size 1) (drill 0.5) (layers F.Cu B.Cu) (net 18))
-  (segment (start 84.75 109.25) (end 86 108) (width 0.35) (layer F.Cu) (net 18))
-  (via (at 86 108) (size 1) (drill 0.5) (layers F.Cu B.Cu) (net 18))
-  (segment (start 83.5 109.25) (end 84.75 109.25) (width 0.35) (layer F.Cu) (net 18))
-  (segment (start 82.25 108) (end 83.5 109.25) (width 0.35) (layer F.Cu) (net 18))
-  (segment (start 82.25 100.5) (end 82.25 108) (width 0.35) (layer F.Cu) (net 18))
-  (via (at 82.25 100.5) (size 1) (drill 0.5) (layers F.Cu B.Cu) (net 18))
   (segment (start 44.75 89.25) (end 47.25 89.25) (width 0.35) (layer B.Cu) (net 19) (status 10))
   (segment (start 88.5 105.5) (end 59.75 105.5) (width 0.35) (layer B.Cu) (net 19))
@@
   (segment (start 198.5 103) (end 210.5 103) (width 0.35) (layer B.Cu) (net 84))
   (segment (start 212.75 105.25) (end 210.5 103) (width 0.35) (layer B.Cu) (net 84))
+  (segment (start 136 98) (end 136 96.75) (width 0.35) (layer F.Cu) (net 85))
+  (segment (start 134.75 99.25) (end 136 98) (width 0.35) (layer F.Cu) (net 85))
+  (segment (start 134.75 108) (end 134.75 99.25) (width 0.35) (layer F.Cu) (net 85))
+  (segment (start 86 108) (end 134.75 108) (width 0.35) (layer B.Cu) (net 85))
+  (via (at 134.75 108) (size 1) (drill 0.5) (layers F.Cu B.Cu) (net 85))
+  (segment (start 84.75 109.25) (end 86 108) (width 0.35) (layer F.Cu) (net 85))
+  (via (at 86 108) (size 1) (drill 0.5) (layers F.Cu B.Cu) (net 85))
+  (segment (start 83.5 109.25) (end 84.75 109.25) (width 0.35) (layer F.Cu) (net 85))
+  (segment (start 82.25 108) (end 83.5 109.25) (width 0.35) (layer F.Cu) (net 85))
+  (segment (start 82.25 100.5) (end 82.25 108) (width 0.35) (layer F.Cu) (net 85))
+  (via (at 82.25 100.5) (size 1) (drill 0.5) (layers F.Cu B.Cu) (net 85))
   (segment (start 71 100.5) (end 82.25 100.5) (width 0.35) (layer B.Cu) (net 85))
   (segment (start 223.5 109.25) (end 223.5 108) (width 0.35) (layer B.Cu) (net 85) (status 10))
@@
   (via (at 112.25 76.75) (size 1) (drill 0.5) (layers F.Cu B.Cu) (net 96))
   (segment (start 112.25 74.25) (end 112.25 76.75) (width 0.35) (layer F.Cu) (net 96) (status 10))
-  (segment (start 106 94.25) (end 107.25 95.5) (width 0.35) (layer B.Cu) (net 96))
-  (segment (start 107.25 95.5) (end 143.5 95.5) (width 0.35) (layer B.Cu) (net 96))
-  (via (at 107.25 95.5) (size 1) (drill 0.5) (layers F.Cu B.Cu) (net 96))
-  (via (at 143.5 95.5) (size 1) (drill 0.5) (layers F.Cu B.Cu) (net 96))
-  (segment (start 73.5 94.25) (end 106 94.25) (width 0.35) (layer B.Cu) (net 96))
-  (via (at 73.5 94.25) (size 1) (drill 0.5) (layers F.Cu B.Cu) (net 96))
-  (segment (start 73.5 101.75) (end 73.5 94.25) (width 0.35) (layer F.Cu) (net 96))
-  (segment (start 72.25 103) (end 73.5 101.75) (width 0.35) (layer F.Cu) (net 96))
   (segment (start 109.75 71.75) (end 221 71.75) (width 0.35) (layer B.Cu) (net 97))
   (segment (start 221 76.75) (end 221 71.75) (width 0.35) (layer B.Cu) (net 97) (status 10))
@@
   (via (at 141 98) (size 1) (drill 0.5) (layers F.Cu B.Cu) (net 112))
   (segment (start 106 98) (end 141 98) (width 0.35) (layer B.Cu) (net 112))
+  (segment (start 106 94.25) (end 107.25 95.5) (width 0.35) (layer B.Cu) (net 113))
+  (segment (start 107.25 95.5) (end 143.5 95.5) (width 0.35) (layer B.Cu) (net 113))
+  (via (at 107.25 95.5) (size 1) (drill 0.5) (layers F.Cu B.Cu) (net 113))
+  (via (at 143.5 95.5) (size 1) (drill 0.5) (layers F.Cu B.Cu) (net 113))
+  (segment (start 73.5 94.25) (end 106 94.25) (width 0.35) (layer B.Cu) (net 113))
+  (via (at 73.5 94.25) (size 1) (drill 0.5) (layers F.Cu B.Cu) (net 113))
+  (segment (start 73.5 101.75) (end 73.5 94.25) (width 0.35) (layer F.Cu) (net 113))
+  (segment (start 72.25 103) (end 73.5 101.75) (width 0.35) (layer F.Cu) (net 113))
   (segment (start 72.25 134.25) (end 72.25 125.5) (width 0.35) (layer B.Cu) (net 113) (status 10))
   (segment (start 107.25 89.25) (end 107.25 95.5) (width 0.35) (layer F.Cu) (net 113) (status 10))
@@
   (via (at 72.25 125.5) (size 1) (drill 0.5) (layers F.Cu B.Cu) (net 113))
   (segment (start 72.25 125.5) (end 72.25 103) (width 0.35) (layer F.Cu) (net 113))
-  (segment (start 101 109.25) (end 112.25 109.25) (width 0.35) (layer B.Cu) (net 113))
-  (segment (start 101 119.25) (end 101 109.25) (width 0.35) (layer F.Cu) (net 113))
-  (via (at 101 109.25) (size 1) (drill 0.5) (layers F.Cu B.Cu) (net 113))
-  (segment (start 87.25 119.25) (end 101 119.25) (width 0.35) (layer B.Cu) (net 113))
-  (via (at 101 119.25) (size 1) (drill 0.5) (layers F.Cu B.Cu) (net 113))
-  (segment (start 86 120.5) (end 87.25 119.25) (width 0.35) (layer B.Cu) (net 113))
-  (segment (start 81 120.5) (end 86 120.5) (width 0.35) (layer B.Cu) (net 113))
-  (segment (start 81 125.5) (end 81 120.5) (width 0.35) (layer F.Cu) (net 113))
-  (via (at 81 120.5) (size 1) (drill 0.5) (layers F.Cu B.Cu) (net 113))
-  (via (at 81 125.5) (size 1) (drill 0.5) (layers F.Cu B.Cu) (net 113))
   (segment (start 78.5 88) (end 78.5 120.5) (width 0.35) (layer F.Cu) (net 114))
   (segment (start 69.75 125.5) (end 69.75 120.5) (width 0.35) (layer F.Cu) (net 114))
@@
   (segment (start 151 94.25) (end 151 101.75) (width 0.35) (layer F.Cu) (net 114) (status 20))
   (segment (start 109.75 99.25) (end 109.75 94.25) (width 0.35) (layer F.Cu) (net 114) (status 10))
+  (segment (start 101 109.25) (end 112.25 109.25) (width 0.35) (layer B.Cu) (net 115))
+  (segment (start 101 119.25) (end 101 109.25) (width 0.35) (layer F.Cu) (net 115))
+  (via (at 101 109.25) (size 1) (drill 0.5) (layers F.Cu B.Cu) (net 115))
+  (segment (start 87.25 119.25) (end 101 119.25) (width 0.35) (layer B.Cu) (net 115))
+  (via (at 101 119.25) (size 1) (drill 0.5) (layers F.Cu B.Cu) (net 115))
+  (segment (start 86 120.5) (end 87.25 119.25) (width 0.35) (layer B.Cu) (net 115))
+  (segment (start 81 120.5) (end 86 120.5) (width 0.35) (layer B.Cu) (net 115))
+  (segment (start 81 125.5) (end 81 120.5) (width 0.35) (layer F.Cu) (net 115))
+  (via (at 81 120.5) (size 1) (drill 0.5) (layers F.Cu B.Cu) (net 115))
+  (via (at 81 125.5) (size 1) (drill 0.5) (layers F.Cu B.Cu) (net 115))
   (segment (start 112.25 109.25) (end 112.25 99.25) (width 0.35) (layer F.Cu) (net 115) (status 20))
   (via (at 112.25 109.25) (size 1) (drill 0.5) (layers F.Cu B.Cu) (net 115))
@@
   (segment (start 57.25 134.25) (end 57.25 124.25) (width 0.35) (layer F.Cu) (net 130) (status 10))
   (via (at 57.25 124.25) (size 1) (drill 0.5) (layers F.Cu B.Cu) (net 130))
+  (zone (net 0) (net_name "") (layer F.Mask) (hatch full 0.508)
+    (connect_pads (clearance 0.508))
+    (min_thickness 0.254)
+    (fill yes (arc_segments 16) (thermal_gap 0.508) (thermal_bridge_width 0.508))
+    (polygon
+      (pts
+        (xy 244.605 117.43) (xy 258.575 117.43) (xy 258.575 121.24) (xy 244.605 121.24)
+      )
+    )
+  )
 )
