File: rk86kngmd.kicad_pcb (KiCad board)
At the start: 2 copper layers, 226.2 x 62.5 mm, 39 parts, among them P1 CONN_01X01, P10 CONN_01X01, P11 CONN_01X01, P12 CONN_01X01, P13 CONN_01X01, P14 CONN_01X01, P2 CONN_01X01, P3 CONN_01X01, P4 CONN_01X01, P5 CONN_01X01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

Commit message: Assy text updated
Parts:
- P1: value CONN_01X01 -> GND
- P10: value CONN_01X01 -> TR00
- P11: value CONN_01X01 -> WPRT
- P12: value CONN_01X01 -> RD_DATA
- P13: value CONN_01X01 -> SIDE
- P14: value CONN_01X01 -> READY
- P2: value CONN_01X01 -> +5V
- P3: value CONN_01X01 -> IP
- P4: value CONN_01X01 -> DISC_A
- P5: value CONN_01X01 -> DISC_B
- P6: value CONN_01X01 -> DIR
- P7: value CONN_01X01 -> STEP
- P8: value CONN_01X01 -> WR_DATA
- P9: value CONN_01X01 -> WR_GATE
